File: stir_plate/stir_plate.kicad_sch (KiCad schematic)
At the start: 11 parts, among them Q1 TIP120, SW1 SW_SPST, U1 LM7805_TO220, U2 ATtiny85-20P, U3 LM3914N

Commit message: updating files
Parts:
- removed SW1: SW_SPST, symbol Switch:SW_SPST
- added C3: 0.1uF, Capacitor_SMD:C_0805_2012Metric_Pad1.18x1.45mm_HandSolder, symbol Device:C
- added D2: LED, LED_THT:LED_D5.0mm, symbol Device:LED
- added PowerIn1: Conn_01x02_Pin, Connector_PinHeader_2.54mm:PinHeader_1x02_P2.54mm_Vertical, symbol Connector:Conn_01x02_Pin
- added R2: 4.7K, Resistor_SMD:R_0805_2012Metric_Pad1.20x1.40mm_HandSolder, symbol Device:R
- added R3: 2.9K, Resistor_SMD:R_0805_2012Metric_Pad1.20x1.40mm_HandSolder, symbol Device:R
- added R4: 1K, Resistor_SMD:R_0805_2012Metric_Pad1.20x1.40mm_HandSolder, symbol Device:R
- added R5: 220 ohm, Resistor_SMD:R_0805_2012Metric_Pad1.20x1.40mm_HandSolder, symbol Device:R
- added SW2: Down, Button_Switch_THT:SW_PUSH_6mm_H5mm, symbol Switch:SW_Push
- added SW3: Up, Button_Switch_THT:SW_PUSH_6mm_H5mm, symbol Switch:SW_Push
- renumbered StirPlatePower to StirPlatePower1
Connections:
- net at C1.1, U1.1 (VI): now also StirPlatePower1.1 (Pin_1), PowerIn1.2 (Pin_2)
- net GND: now reaches C1.2, C2.1, D1.2 (A), Q1.3 (E), U1.2 (GND), U2.4 (GND), U3.2 (V-), U3.4 (RLO)
- net GND: now also C3.2, R3.1, R5.1, SW2.2, SW3.1
- net at U2.5 (AREF/PB0): now also R2.2; no longer R1.2
- net at U2.2 (XTAL1/PB3): now also SW2.1
- net at U2.3 (XTAL2/PB4): now also SW3.2
- net at U2.6 (PB1): now also R1.2
- net at U2.7 (PB2): now also D2.2 (A)
- net at U3.5 (SIG): now also C3.1, R2.1
- net at U3.6 (RHI): now also U3.7 (REFOUT), R4.2
- net at U3.8 (REFADJ): now also R3.2, R4.1
- new net: D2.1 (K), R5.2
- new net +12P: PowerIn1.1 (Pin_1)
Other:
- moved on the sheet: BAR1, U3
